Commit message: feat: tool added

File: robots/panda.gazebo.xacro (robot description, xacro)
@@ -1,5 +1,5 @@
 <?xml version="1.0"?>
 <robot xmlns:xacro="http://www.ros.org/wiki/xacro">
-    <xacro:macro name="panda_gazebo" params="robot_name load_gripper">
+    <xacro:macro name="panda_gazebo" params="robot_name">
         <gazebo reference="${robot_name}_link0">
             <material>Gazebo/Grey</material>
@@ -55,62 +55,36 @@
             <mu2>0.2</mu2>
         </gazebo>
-        <!-- LinkHand -->
-        <gazebo reference="${robot_name}_hand">
-            <material>Gazebo/Grey</material>
-            <mu1>0.2</mu1>
-            <mu2>0.2</mu2>
+        <gazebo reference="${robot_name}_joint1">
+          <implicitSpringDamper>1</implicitSpringDamper>
+          <provideFeedback>true</provideFeedback>
         </gazebo>
-        <xacro:if value="${load_gripper}">
-            <!-- LinkRightFinger -->
-            <gazebo reference="${robot_name}_rightfinger">
-                <material>Gazebo/Grey</material>
-                <mu1>0.2</mu1>
-                <mu2>0.2</mu2>
-            </gazebo>
-            <!-- LinkLeftFinger -->
-            <gazebo reference="${robot_name}_leftfinger">
-                <material>Gazebo/Grey</material>
-                <mu1>0.2</mu1>
-                <mu2>0.2</mu2>
-            </gazebo>
-        </xacro:if>
-      <gazebo reference="${robot_name}_joint7">
-        <implicitSpringDamper>1</implicitSpringDamper>
-        <provideFeedback>true</provideFeedback>
-      </gazebo>
-      <gazebo reference="${robot_name}_joint1">
-        <implicitSpringDamper>1</implicitSpringDamper>
-        <provideFeedback>true</provideFeedback>
-      </gazebo>
-      <gazebo reference="${robot_name}_joint2">
-        <implicitSpringDamper>1</implicitSpringDamper>
-        <provideFeedback>true</provideFeedback>
-      </gazebo>
-      <gazebo reference="${robot_name}_joint3">
-        <implicitSpringDamper>1</implicitSpringDamper>
-        <provideFeedback>true</provideFeedback>
-      </gazebo>
-      <gazebo reference="${robot_name}_joint4">
-        <implicitSpringDamper>1</implicitSpringDamper>
-        <provideFeedback>true</provideFeedback>
-      </gazebo>
-      <gazebo reference="${robot_name}_joint5">
-        <implicitSpringDamper>1</implicitSpringDamper>
-        <provideFeedback>true</provideFeedback>
-      </gazebo>
-      <gazebo reference="${robot_name}_joint6">
-        <implicitSpringDamper>1</implicitSpringDamper>
-        <provideFeedback>true</provideFeedback>
-      </gazebo>
-      <xacro:if value="${load_gripper}">
-          <gazebo reference="${robot_name}_finger_joint1">
-            <implicitSpringDamper>1</implicitSpringDamper>
-            <provideFeedback>true</provideFeedback>
-          </gazebo>
-          <gazebo reference="${robot_name}_finger_joint2">
-            <implicitSpringDamper>1</implicitSpringDamper>
-            <provideFeedback>true</provideFeedback>
-          </gazebo>
-      </xacro:if>
+        <gazebo reference="${robot_name}_joint2">
+          <implicitSpringDamper>1</implicitSpringDamper>
+          <provideFeedback>true</provideFeedback>
+        </gazebo>
+        <gazebo reference="${robot_name}_joint3">
+          <implicitSpringDamper>1</implicitSpringDamper>
+          <provideFeedback>true</provideFeedback>
+        </gazebo>
+        <gazebo reference="${robot_name}_joint4">
+          <implicitSpringDamper>1</implicitSpringDamper>
+          <provideFeedback>true</provideFeedback>
+        </gazebo>
+        <gazebo reference="${robot_name}_joint5">
+          <implicitSpringDamper>1</implicitSpringDamper>
+          <provideFeedback>true</provideFeedback>
+        </gazebo>
+        <gazebo reference="${robot_name}_joint6">
+          <implicitSpringDamper>1</implicitSpringDamper>
+          <provideFeedback>true</provideFeedback>
+        </gazebo>
+        <gazebo reference="${robot_name}_joint7">
+          <implicitSpringDamper>1</implicitSpringDamper>
+          <provideFeedback>true</provideFeedback>
+        </gazebo>
+        <gazebo reference="${robot_name}_joint8">
+          <implicitSpringDamper>1</implicitSpringDamper>
+          <provideFeedback>true</provideFeedback>
+        </gazebo>
     </xacro:macro>
 </robot>

File: robots/panda.transmission.xacro (robot description, xacro)
@@ -1,13 +1,7 @@
 <?xml version="1.0"?>
 <robot xmlns:xacro="http://www.ros.org/wiki/xacro">
-    <xacro:macro name="panda_transmission" params="robot_name load_gripper">
+    <xacro:macro name="panda_transmission" params="robot_name">
         <!-- Load Gazebo lib and set the robot namespace -->
         <gazebo>
-            <!--plugin name="panda_ros_control" filename="libpanda_gazebo_ros_control.so">
-                <robotNamespace></robotNamespace>
-                <robotSimType>panda_gazebo/PandaRobotHWSim</robotSimType>
-                <controlPeriod>0.001</controlPeriod>
-                <eStopTopic>sim_estop</eStopTopic>
-            </plugin-->
             <plugin name="gazebo_ros_control" filename="libgazebo_ros_control.so">
                 <robotNamespace>/panda</robotNamespace>
@@ -86,26 +80,4 @@
             </actuator>
         </transmission>
-        <xacro:if value="${load_gripper}">
-            <transmission name="${robot_name}_leftfinger">
-                <type>transmission_interface/SimpleTransmission</type>
-                <joint name="${robot_name}_finger_joint1">
-                    <hardwareInterface>hardware_interface/EffortJointInterface</hardwareInterface>
-                </joint>
-                <actuator name="${robot_name}_finger_joint1">
-                    <hardwareInterface>hardware_interface/EffortJointInterface</hardwareInterface>
-                    <mechanicalReduction>1</mechanicalReduction>
-                </actuator>
-            </transmission>
-            <transmission name="${robot_name}_rightfinger">
-                <type>transmission_interface/SimpleTransmission</type>
-                <joint name="${robot_name}_finger_joint2">
-                    <hardwareInterface>hardware_interface/EffortJointInterface</hardwareInterface>
-                </joint>
-                <actuator name="${robot_name}_finger_joint2">
-                    <hardwareInterface>hardware_interface/EffortJointInterface</hardwareInterface>
-                    <mechanicalReduction>1</mechanicalReduction>
-                </actuator>
-            </transmission>
-        </xacro:if>
     </xacro:macro>
 </robot>

File: robots/panda_arm.urdf (robot description, URDF)
Before this commit: robot panda, 9 links, 8 joints
Links:
- link panda_link8: geometry collision mesh filename=meshes/collision/tool.stl; visual mesh filename=meshes/visual/tool.dae

File: robots/panda_arm.xacro (robot description, xacro)
@@ -1,5 +1,5 @@
 <?xml version='1.0'?>
 <robot xmlns:xacro="http://www.ros.org/wiki/xacro" name="panda">
-  <xacro:macro name="panda_arm" params="arm_id:='panda' description_pkg:='franka_description' connected_to:=''  in_gazebo='false' xyz:='0 0 0' rpy:='0 0 0'">
+  <xacro:macro name="panda_arm" params="arm_id:='panda' description_pkg:='franka_panda_description' connected_to:=''  in_gazebo='false' xyz:='0 0 0' rpy:='0 0 0'">
     <xacro:unless value="${not connected_to}">
       <joint name="${arm_id}_joint_${connected_to}" type="fixed">
@@ -221,4 +221,14 @@
     </joint>
     <link name="${arm_id}_link8">
+      <visual>
+        <geometry>
+          <mesh filename="package://franka_panda_description/meshes/visual/tool.dae"/>
+        </geometry>
+      </visual>
+      <collision>
+        <geometry>
+          <mesh filename="package://franka_panda_description/meshes/collision/tool.stl"/>
+        </geometry>
+      </collision>
       <inertial>
         <origin xyz="0 0 0" rpy="0 0 0"/>

File: robots/panda_arm_hand.urdf.xacro (robot description, xacro)
@@ -2,25 +2,15 @@
 <robot xmlns:xacro="http://www.ros.org/wiki/xacro" name="panda">
   <xacro:arg name="robot_name" default="panda"/>
-  <xacro:arg name="load_tool" default="false"/>
-  <xacro:arg name="load_gripper" default="false"/>
   <xacro:arg name="load_gazebo" default="false"/>
   <xacro:include filename="$(find franka_panda_description)/robots/panda_arm.xacro"/>
-  <!--xacro:if value="$(arg load_tool)">
-    <xacro:include filename="$(find franka_panda_description)/robots/tool.xacro"/>
-    <xacro:tool ns="panda" rpy="0 0 ${-pi/4}" connected_to="panda_link8"/>
-  </xacro:if>
-  <xacro:if value="$(arg load_gripper)">
-    <xacro:include filename="$(find franka_panda_description)/robots/hand.xacro"/>
-    <xacro:hand ns="panda" rpy="0 0 ${-pi/4}" connected_to="panda_link8"/>
-  </xacro:if-->
+  <xacro:unless value="$(arg load_gazebo)">
+    <xacro:panda_arm />
+  </xacro:unless>
   <xacro:if value="$(arg load_gazebo)">
     <xacro:include filename="$(find franka_panda_description)/robots/panda.gazebo.xacro"/>
     <xacro:include filename="$(find franka_panda_description)/robots/panda.transmission.xacro"/>
     <xacro:panda_arm in_gazebo="true" />
-    <xacro:panda_gazebo robot_name="$(arg robot_name)" load_gripper="$(arg load_gripper)"/>
-    <xacro:panda_transmission robot_name="$(arg robot_name)" load_gripper="$(arg load_gripper)"/>
+    <xacro:panda_gazebo robot_name="$(arg robot_name)"/>
+    <xacro:panda_transmission robot_name="$(arg robot_name)"/>
   </xacro:if>
-  <xacro:unless value="$(arg load_gazebo)">
-    <xacro:panda_arm />
-  </xacro:unless>
 </robot>
